Commit message: 10th March

File: src/my_robot_description/urdf/mobile_base_gazebo.xacro (robot description, xacro)
@@ -2,14 +2,14 @@
 <robot xmlns:xacro="http://www.ros.org/wiki/xacro">
     <gazebo reference="base_link">
-        <material>Gazebo/Blue</material>
+        <material>Gazebo/Orange</material>
     </gazebo>
     <gazebo reference="right_wheel_link">
-        <material>Gazebo/Grey</material>
+        <material>Gazebo/Red</material>
     </gazebo>
     <gazebo reference="left_wheel_link">
-        <material>Gazebo/Grey</material>
+        <material>Gazebo/Red</material>
     </gazebo>
     <gazebo reference="caster_wheel_link">
-        <material>Gazebo/Grey</material>
+        <material>Gazebo/Indigo</material>
         <mu1 value="0.1" />
         <mu2 value="0.1" />
