Commit message: 16th March

File: src/my_robot_description/urdf/camera.xacro (robot description, xacro)
@@ -9,5 +9,5 @@
                 <box size="${camera_length} ${camera_width} ${camera_height}"/>
             </geometry>
-            <material name="grey" />
+            <material name="blue" />
         </visual>
         <collision>

File: src/my_robot_description/urdf/common_properties.xacro (robot description, xacro)
@@ -4,6 +4,18 @@
         <color rgba="0 0 0.5 1" />
     </material>
-    <material name="grey">
-        <color rgba="0.5 0.5 0.5 1" />
+    <material name="indigo">
+        <color rgba="0.5 0 1.0 1" />
+    </material>
+    <material name="orange">
+        <color rgba="1.0 0.5 0 1"/>
+    </material>
+    <material name="yellow">
+        <color rgba="1.0 1.0 0 1"/>
+    </material>
+    <material name="red">
+        <color rgba="1.0 0 0 1"/>
+    </material>
+    <material name="green">
+        <color rgba="0 1.0 0 1"/>
     </material>
     <xacro:macro name="box_inertia" params="m l w h xyz rpy">

File: src/my_robot_description/urdf/mobile_base.xacro (robot description, xacro)
@@ -13,5 +13,5 @@
             </geometry>
             <origin xyz="0 0 ${base_height / 2.0}" rpy="0 0 0" />
-            <material name="blue" />
+            <material name="orange" />
         </visual>
         <collision>
@@ -31,5 +31,5 @@
                 </geometry>
                 <origin xyz="0 0 0" rpy="${pi / 2.0} 0 0" />
-                <material name="grey" />
+                <material name="red" />
             </visual>
             <collision>
@@ -51,5 +51,5 @@
             </geometry>
             <origin xyz="0 0 0" rpy="0 0 0" />
-            <material name="grey" />
+            <material name="indigo" />
         </visual>
         <collision>

File: src/my_robot_description/urdf/my_robot.urdf.xacro (robot description, xacro)
@@ -4,4 +4,11 @@
     <xacro:include filename="mobile_base.xacro" />
     <xacro:include filename="mobile_base_gazebo.xacro" />
+    <xacro:include filename="arm.xacro" />
+    <xacro:include  filename="arm_gazebo.xacro"/>
+    <joint name="mobile_base_arm_joint" type="fixed">
+        <parent link="base_link"/>
+        <child link="arm_base_link"/>
+        <origin xyz="${base_length / 4.0} 0 ${base_height}" rpy="0 0 0" />
+    </joint>
     <xacro:include filename="camera.xacro" />
 </robot>
